File: CableTester_Logic.kicad_pcb (KiCad board)
At the start: 2 copper layers, 105.7 x 85.9 mm, 29 parts, among them J1 Power, J10 Conn_Coaxial, J11 Conn_Coaxial, J12 Conn_Coaxial, J13 Conn_Coaxial, J14 Conn_Coaxial, J15 Conn_Coaxial, J16 Conn_Coaxial, J17 Conn_Coaxial, J18 Conn_Coaxial, J19 Conn_Coaxial, J2 PWM, J20 MircoMatch -8, J21 MircoMatch -8, J3 Analog, J4 PWM, J5 Analog, J6 Communication, J7 Digital, J8 Conn_Coaxial, J9 Conn_Coaxial, U1 DG1206EUI+, U2 DG1206EUI+

Commit message: Finalized Project for Test Production
Parts:
- added C1: 100nF, Capacitor_SMD:C_0805_2012Metric_Pad1.18x1.45mm_HandSolder, F.Cu at (187.1, 68.5)
- added C2: 100nF, Capacitor_SMD:C_0805_2012Metric_Pad1.18x1.45mm_HandSolder, F.Cu at (187.1, 84.0)
- added MTG1: Conn_02x02_Counter_Clockwise, Project_Footprints:KEYSTONE_7693-5, F.Cu at (108.9, 39.0)
- added MTG2: Conn_02x02_Counter_Clockwise, Project_Footprints:KEYSTONE_7693-5, F.Cu at (108.9, 107.6)
- added MTG3: Conn_02x02_Counter_Clockwise, Project_Footprints:KEYSTONE_7693-5, F.Cu at (195.2, 107.6)
- added MTG4: Conn_02x02_Counter_Clockwise, Project_Footprints:KEYSTONE_7693-5, F.Cu at (195.2, 39.0)
- moved U2 27.2 mm to (181.3, 80.7), turned to 180 degrees
- moved U1 27.1 mm to (181.3, 65.4), turned to 180 degrees
- moved J20 8.15 mm to (209.2, 43.5)
- moved J21 8.15 mm to (209.2, 112.1)
Connections:
- net /*10 renamed /D10
- net /*11 renamed /D11
- net /*12 renamed /D12
- net /*13 renamed /D13
- net /*2 renamed /D2
- net /*3 renamed /D3
- net /*4 renamed /D4
- net /*5 renamed /D5
- net /*52 renamed /SCK/D52
- net /*6 renamed /D6
- net /*7 renamed /D7
- net /*8 renamed /D8
- net /*9 renamed /D9
- net /22 renamed /D22
- net /23 renamed /D23
- net /24 renamed /SCL1/D24
- net /25 renamed /SDA1/D25
- net /36 renamed /D36
- net /37 renamed /D37
- net /48 renamed /D48
- net /49 renamed /D49
- net /50 renamed /MISO/D50
- net /51 renamed /MOSI/D51
- net /53 renamed /SS/D53
- net /RX0/0 renamed /RX/D0
- net /RX1/19 renamed /RX1/D19
- net /RX3/15 renamed /RX3/D15
- net /TX0/1 renamed /TX/D1
- net /TX1/18 renamed /TX1/D18
- net /TX3/14 renamed /TX3/D14
- J10 pad 1: unconnected-(J10-In-Pad1) -> Net-(J10-In)
- J10 pad 2: Net-(J10-Ext-Pad2) -> GND
- J11 pad 1: unconnected-(J11-In-Pad1) -> Net-(J11-In)
- J11 pad 2: Net-(J11-Ext-Pad2) -> GND
- J12 pad 1: unconnected-(J12-In-Pad1) -> Net-(J12-In)
- J12 pad 2: Net-(J12-Ext-Pad2) -> GND
- J13 pad 1: unconnected-(J13-In-Pad1) -> Net-(J13-In)
- J13 pad 2: Net-(J13-Ext-Pad2) -> GND
- J14 pad 1: unconnected-(J14-In-Pad1) -> Net-(J14-In)
- J14 pad 2: Net-(J14-Ext-Pad2) -> GND
- J15 pad 1: unconnected-(J15-In-Pad1) -> Net-(J15-In)
- J15 pad 2: Net-(J15-Ext-Pad2) -> GND
- J16 pad 1: unconnected-(J16-In-Pad1) -> Net-(J16-In)
- J16 pad 2: Net-(J16-Ext-Pad2) -> GND
- J17 pad 1: unconnected-(J17-In-Pad1) -> Net-(J17-In)
- J17 pad 2: Net-(J17-Ext-Pad2) -> GND
- J18 pad 1: unconnected-(J18-In-Pad1) -> Net-(J18-In)
- J18 pad 2: Net-(J18-Ext-Pad2) -> GND
- J19 pad 1: unconnected-(J19-In-Pad1) -> Net-(J19-In)
- J19 pad 2: Net-(J19-Ext-Pad2) -> GND
- J20 pad 1: unconnected-(J20-Pad1) -> +5V
- J20 pad 2: unconnected-(J20-Pad2) -> +3V3
- J20 pad 3: unconnected-(J20-Pad3) -> /D27
- J20 pad 4: unconnected-(J20-Pad4) -> /D33
- J20 pad 5: unconnected-(J20-Pad5) -> /D29
- J20 pad 6: unconnected-(J20-Pad6) -> /D35
- J20 pad 7: unconnected-(J20-Pad7) -> /D31
- J20 pad 8: unconnected-(J20-Pad8) -> GND
- J21 pad 1: unconnected-(J21-Pad1) -> +5V
- J21 pad 2: unconnected-(J21-Pad2) -> +3V3
- J21 pad 3: unconnected-(J21-Pad3) -> /D43
- J21 pad 4: unconnected-(J21-Pad4) -> /D39
- J21 pad 5: unconnected-(J21-Pad5) -> /D45
- J21 pad 6: unconnected-(J21-Pad6) -> /D41
- J21 pad 7: unconnected-(J21-Pad7) -> /D47
- J21 pad 8: unconnected-(J21-Pad8) -> GND
- J6 pad 3: /TX2/16 -> /TX2/D16
- J6 pad 4: /RX2/17 -> /RX2/D17
- J6 pad 7: /SDA/20 -> /SDA/D20
- J6 pad 8: /SCL/21 -> /SCL/D21
- J7 pad 10: /47 -> /D47
- J7 pad 11: /*44 -> /D44
- J7 pad 12: /*45 -> /D45
- J7 pad 13: /42 -> /D42
- J7 pad 14: /43 -> /D43
- J7 pad 15: /40 -> /D40
- J7 pad 16: /41 -> /D41
- J7 pad 17: /38 -> /D38
- J7 pad 18: /39 -> /D39
- J7 pad 21: /34 -> /D34
- J7 pad 22: /35 -> /D35
- J7 pad 23: /32 -> /D32
- J7 pad 24: /33 -> /D33
- J7 pad 25: /30 -> /D30
- J7 pad 26: /31 -> /D31
- J7 pad 27: /28 -> /D28
- J7 pad 28: /29 -> /D29
- J7 pad 29: /26 -> /D26
- J7 pad 30: /27 -> /D27
- J7 pad 9: /*46 -> /D46
- J8 pad 1: unconnected-(J8-In-Pad1) -> Net-(J8-In)
- J8 pad 2: Net-(J8-Ext-Pad2) -> GND
- J9 pad 1: unconnected-(J9-In-Pad1) -> Net-(J9-In)
- J9 pad 2: Net-(J9-Ext-Pad2) -> GND
- U1 pad 1: unconnected-(U1-VPOS-Pad1) -> +5V
- U1 pad 12: unconnected-(U1-GND-Pad12) -> GND
- U1 pad 14: unconnected-(U1-A3-Pad14) -> /D34
- U1 pad 15: unconnected-(U1-A2-Pad15) -> /D26
- U1 pad 16: unconnected-(U1-A1-Pad16) -> /D28
- U1 pad 17: unconnected-(U1-A0-Pad17) -> /D30
- U1 pad 18: unconnected-(U1-EN-Pad18) -> /D32
- U1 pad 19: unconnected-(U1-NO1-Pad19) -> Net-(J8-In)
- U1 pad 20: unconnected-(U1-NO2-Pad20) -> Net-(J9-In)
- U1 pad 21: unconnected-(U1-NO3-Pad21) -> Net-(J10-In)
- U1 pad 22: unconnected-(U1-NO4-Pad22) -> Net-(J11-In)
- U1 pad 23: unconnected-(U1-NO5-Pad23) -> Net-(J12-In)
- U1 pad 24: unconnected-(U1-NO6-Pad24) -> Net-(J13-In)
- U1 pad 27: unconnected-(U1-VNEG-Pad27) -> GND
- U1 pad 28: unconnected-(U1-COM-Pad28) -> /TX2/D16
- U2 pad 1: unconnected-(U2-VPOS-Pad1) -> +5V
- U2 pad 12: unconnected-(U2-GND-Pad12) -> GND
- U2 pad 14: unconnected-(U2-A3-Pad14) -> /D46
- U2 pad 15: unconnected-(U2-A2-Pad15) -> /D38
- U2 pad 16: unconnected-(U2-A1-Pad16) -> /D40
- U2 pad 17: unconnected-(U2-A0-Pad17) -> /D42
- U2 pad 18: unconnected-(U2-EN-Pad18) -> /D44
- U2 pad 19: unconnected-(U2-NO1-Pad19) -> Net-(J19-In)
- U2 pad 20: unconnected-(U2-NO2-Pad20) -> Net-(J18-In)
- U2 pad 21: unconnected-(U2-NO3-Pad21) -> Net-(J17-In)
- U2 pad 22: unconnected-(U2-NO4-Pad22) -> Net-(J16-In)
- U2 pad 23: unconnected-(U2-NO5-Pad23) -> Net-(J15-In)
- U2 pad 24: unconnected-(U2-NO6-Pad24) -> Net-(J14-In)
- U2 pad 27: unconnected-(U2-VNEG-Pad27) -> GND
- U2 pad 28: unconnected-(U2-COM-Pad28) -> /RX2/D17
Routing:
- net +5V: track 0.00 -> 272.3 mm, vias 0 -> 4
- net +3V3: track 0.00 -> 206.2 mm, vias 0 -> 2
- net Net-(J13-In): track 0.00 -> 81.0 mm
- net Net-(J19-In): track 0.00 -> 75.9 mm
- net Net-(J12-In): track 0.00 -> 69.1 mm
- net Net-(J18-In): track 0.00 -> 62.3 mm
- net Net-(J11-In): track 0.00 -> 55.5 mm
- net Net-(J17-In): track 0.00 -> 49.5 mm
- net /D39: track 0.00 -> 45.4 mm
- net Net-(J10-In): track 0.00 -> 40.0 mm
- net /D35: track 0.00 -> 39.7 mm
- net /RX2/D17: track 0.00 -> 39.5 mm, vias 0 -> 1
- net /D41: track 0.00 -> 39.4 mm
- net /D43: track 0.00 -> 38.8 mm
- net Net-(J16-In): track 0.00 -> 38.6 mm
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- added copper zone on B.Cu, net GND
Other:
- board size 105.7 x 85.9 mm -> 110.7 x 85.9 mm
- board text added: "ALS-U Controls Cable Tester Logic Pedro Rodriguez Rev 1.0 - beta"
- board text removed: "ALS-U Controls Cable Tester Logic Pedro Rodriguez"
